File: kicad/voltagerecorder/voltage_input.kicad_sch (KiCad schematic)
At the start: 12 parts

Commit message: a
Parts:
- U1: renamed from U?; footprint (none) -> Package_SO:TSSOP-14_4.4x5mm_P0.65mm
- gave numbers to parts that had none: 11
Changed lines of the file:
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@@
   (symbol (lib_id "power:+12V") (at 135.89 78.74 0) (unit 1)
     (in_bom yes) (on_board yes) (fields_autoplaced)
-    (property "Reference" "#PWR?" (id 0) (at 135.89 82.55 0)
+    (property "Reference" "#PWR056" (id 0) (at 135.89 82.55 0)
       (effects (font (size 1.27 1.27)) hide)
     )
@@
   (symbol (lib_id "Device:C") (at 119.38 100.33 0) (unit 1)
     (in_bom yes) (on_board yes) (fields_autoplaced)
-    (property "Reference" "C?" (id 0) (at 123.19 99.0599 0)
+    (property "Reference" "C27" (id 0) (at 123.19 99.0599 0)
       (effects (font (size 1.27 1.27)) (justify left))
     )
@@
   (symbol (lib_id "Device:Opamp_Quad") (at 171.45 95.25 0) (unit 1)
     (in_bom yes) (on_board yes) (fields_autoplaced)
-    (property "Reference" "U?" (id 0) (at 171.45 85.09 0))
+    (property "Reference" "U1" (id 0) (at 171.45 85.09 0))
     (property "Value" "Opamp_Quad" (id 1) (at 171.45 87.63 0))
-    (property "Footprint" "" (id 2) (at 171.45 95.25 0)
+    (property "Footprint" "Package_SO:TSSOP-14_4.4x5mm_P0.65mm" (id 2) (at 171.45 95.25 0)
       (effects (font (size 1.27 1.27)) hide)
     )
@@
   (symbol (lib_id "Device:R") (at 170.18 105.41 90) (unit 1)
     (in_bom yes) (on_board yes)
-    (property "Reference" "R?" (id 0) (at 170.18 107.95 90))
+    (property "Reference" "R30" (id 0) (at 170.18 107.95 90))
     (property "Value" "100" (id 1) (at 170.18 110.49 90))
     (property "Footprint" "" (id 2) (at 170.18 107.188 90)
@@
   (symbol (lib_id "power:-12V") (at 135.89 106.68 180) (unit 1)
     (in_bom yes) (on_board yes) (fields_autoplaced)
-    (property "Reference" "#PWR?" (id 0) (at 135.89 109.22 0)
+    (property "Reference" "#PWR057" (id 0) (at 135.89 109.22 0)
       (effects (font (size 1.27 1.27)) hide)
     )
@@
   (symbol (lib_id "power:GND") (at 195.58 106.68 0) (unit 1)
     (in_bom yes) (on_board yes) (fields_autoplaced)
-    (property "Reference" "#PWR?" (id 0) (at 195.58 113.03 0)
+    (property "Reference" "#PWR058" (id 0) (at 195.58 113.03 0)
       (effects (font (size 1.27 1.27)) hide)
     )
@@
   (symbol (lib_id "Connector:Conn_01x01_Male") (at 147.32 87.63 270) (unit 1)
     (in_bom yes) (on_board yes)
-    (property "Reference" "J?" (id 0) (at 148.59 86.9949 90)
+    (property "Reference" "J7" (id 0) (at 148.59 86.9949 90)
       (effects (font (size 1.27 1.27)) (justify left))
     )
@@
   (symbol (lib_id "Device:R") (at 187.96 95.25 90) (unit 1)
     (in_bom yes) (on_board yes)
-    (property "Reference" "R?" (id 0) (at 187.96 97.79 90))
+    (property "Reference" "R31" (id 0) (at 187.96 97.79 90))
     (property "Value" "100" (id 1) (at 187.96 100.33 90))
     (property "Footprint" "" (id 2) (at 187.96 97.028 90)
@@
   (symbol (lib_id "power:GND") (at 106.68 106.68 0) (unit 1)
     (in_bom yes) (on_board yes) (fields_autoplaced)
-    (property "Reference" "#PWR?" (id 0) (at 106.68 113.03 0)
+    (property "Reference" "#PWR054" (id 0) (at 106.68 113.03 0)
       (effects (font (size 1.27 1.27)) hide)
     )
@@
   (symbol (lib_id "Device:C") (at 195.58 101.6 0) (unit 1)
     (in_bom yes) (on_board yes) (fields_autoplaced)
-    (property "Reference" "C?" (id 0) (at 199.39 100.3299 0)
+    (property "Reference" "C28" (id 0) (at 199.39 100.3299 0)
       (effects (font (size 1.27 1.27)) (justify left))
     )
@@
   (symbol (lib_id "Device:R") (at 87.63 92.71 90) (unit 1)
     (in_bom yes) (on_board yes)
-    (property "Reference" "R?" (id 0) (at 87.63 87.63 90))
+    (property "Reference" "R26" (id 0) (at 87.63 87.63 90))
     (property "Value" "330k" (id 1) (at 87.63 90.17 90))
     (property "Footprint" "" (id 2) (at 87.63 94.488 90)
@@
   (symbol (lib_id "Device:D_Dual_Series_KAC") (at 135.89 92.71 90) (unit 1)
     (in_bom yes) (on_board yes)
-    (property "Reference" "D?" (id 0) (at 140.97 80.01 90)
+    (property "Reference" "D4" (id 0) (at 140.97 80.01 90)
       (effects (font (size 1.27 1.27)) (justify left))
     )
@@
   (symbol (lib_id "power:GND") (at 119.38 106.68 0) (unit 1)
     (in_bom yes) (on_board yes) (fields_autoplaced)
-    (property "Reference" "#PWR?" (id 0) (at 119.38 113.03 0)
+    (property "Reference" "#PWR055" (id 0) (at 119.38 113.03 0)
       (effects (font (size 1.27 1.27)) hide)
     )
@@
   (symbol (lib_id "Device:R") (at 156.21 92.71 270) (unit 1)
     (in_bom yes) (on_board yes)
-    (property "Reference" "R?" (id 0) (at 154.94 88.9 0))
+    (property "Reference" "R29" (id 0) (at 154.94 88.9 0))
     (property "Value" "1k" (id 1) (at 157.48 88.9 0))
     (property "Footprint" "" (id 2) (at 156.21 90.932 90)
@@
   (symbol (lib_id "Device:R") (at 78.74 92.71 90) (unit 1)
     (in_bom yes) (on_board yes)
-    (property "Reference" "R?" (id 0) (at 78.74 87.63 90))
+    (property "Reference" "R25" (id 0) (at 78.74 87.63 90))
     (property "Value" "330k" (id 1) (at 78.74 90.17 90))
     (property "Footprint" "" (id 2) (at 78.74 94.488 90)
@@
   (symbol (lib_id "Device:R") (at 106.68 100.33 180) (unit 1)
     (in_bom yes) (on_board yes)
-    (property "Reference" "R?" (id 0) (at 110.49 99.06 0))
+    (property "Reference" "R28" (id 0) (at 110.49 99.06 0))
     (property "Value" "10k" (id 1) (at 110.49 101.6 0))
     (property "Footprint" "" (id 2) (at 108.458 100.33 90)
@@
   (symbol (lib_id "Device:R") (at 96.52 92.71 90) (unit 1)
     (in_bom yes) (on_board yes)
-    (property "Reference" "R?" (id 0) (at 96.52 87.63 90))
+    (property "Reference" "R27" (id 0) (at 96.52 87.63 90))
     (property "Value" "330k" (id 1) (at 96.52 90.17 90))
     (property "Footprint" "" (id 2) (at 96.52 94.488 90)

Commit message: Footprints komplett zugeordnet.
Parts:
- removed C28: 15n, symbol Device:C
- removed D4: D_Dual_Series_KAC, symbol Device:D_Dual_Series_KAC
- added D4: BAV99, Package_TO_SOT_SMD:SOT-23, symbol Diode:BAV99
- C27: footprint (none) -> Capacitor_SMD:C_0603_1608Metric_Pad1.08x0.95mm_HandSolder
- J7: footprint (none) -> Connector_PinHeader_2.54mm:PinHeader_1x01_P2.54mm_Vertical
- R25, R26, R27: footprint (none) -> Resistor_SMD:R_MELF_MMB-0207
- R28: footprint (none) -> Resistor_SMD:R_1206_3216Metric_Pad1.30x1.75mm_HandSolder
- R29, R30: footprint (none) -> Resistor_SMD:R_0603_1608Metric_Pad0.98x0.95mm_HandSolder
- R31: value 100 -> 470; footprint (none) -> Resistor_SMD:R_0603_1608Metric_Pad0.98x0.95mm_HandSolder
Connections:
- net +12V: now also D4.2 (A)
- net -12V: now also D4.1 (K)
- net at C27.1, J7.1 (Pin_1), R27.2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: now also D4.3 (K)
Other:
- note removed: "106kHz"
