File: kicad/voltagerecorder/voltagerecorder.kicad_sch (KiCad schematic)
At the start: 82 parts, among them J1 Conn_02x10_Odd_Even, J3 Conn_01x08, P1 DM3CS-SF, U1 Opamp_Quad, U5 ADS8638, U8 ESP32-C3-WROOM-02

Commit message: pins zugeordnet
Parts:
- removed R3: nc, Resistor_SMD:R_0603_1608Metric_Pad0.98x0.95mm_HandSolder, symbol Device:R
- removed R36, R37: 10k, Resistor_SMD:R_0603_1608Metric_Pad0.98x0.95mm_HandSolder, symbol Device:R
- added J?: Conn_01x06, symbol Connector_Generic:Conn_01x06
- added R? (x2): 1k, Resistor_SMD:R_0603_1608Metric_Pad0.98x0.95mm_HandSolder, symbol Device:R
- added R? (x2): 10k, Resistor_SMD:R_0603_1608Metric_Pad0.98x0.95mm_HandSolder, symbol Device:R
- R?: value 100k -> 10k
Connections:
- net RAM_CLK is gone; now on net SPI2_SCK: U?.6 (SCLK)
- net RAM_CS is gone; now on net SPI2_NSS: U?.1 (~{CE})
- net RAM_SIO0 is gone; now on net SPI2_MISO: U?.2 (SO/SIO)
- net RAM_SIO1 is gone; now on net SPI2_MOSI: U?.5 (SI/SIO)
- net +3.3V: now also U8.1 (3V3), U8.7 (GPIO8), R?.2, R?.2
- net CS: no longer R2.1, U5.16 (CS)
- net GND: now also U8.10 (GPIO10), J?.6 (Pin_6)
- net MISO: no longer R1.2
- net MOSI: no longer U5.18 (DIN)
- net SCLK: no longer U5.17 (SCLK)
- net USB_CC1: no longer U?.41 (PB4), U?.42 (PB5)
- net USB_CC2: no longer U?.43 (PB6), U?.44 (PB7)
- net SPI3_SCK: now reaches P1.5 (CLK), R34.1
- net SPI3_SCK: now also U?.40 (PB3)
- net UART_G4TX_ESPRX: now reaches U8.11 (GPIO20/U0RXD)
- net UART_G4TX_ESPRX: now also J?.5 (Pin_5), R?.2
- net UART_G4RX_ESPTX: now reaches U8.12 (GPIO21/U0TXD)
- net UART_G4RX_ESPTX: now also J?.4 (Pin_4), R?.2
- net ESP_EN: now reaches U8.2 (EN/CHIP_PU)
- net ESP_EN: now also J?.2 (Pin_2), R?.1
- net ESP_BOOT: now reaches U8.8 (GPIO9)
- net ESP_BOOT: now also J?.3 (Pin_3), R?.1
- net SENSE_+5V: now reaches C38.1, R39.1, R40.2
- net SPI3_MOSI: now reaches P1.3 (CMD), R33.1
- net SPI3_MOSI: now also U?.42 (PB5)
- net SPI3_MISO: now reaches P1.7 (DAT0), R35.1
- net SPI3_MISO: now also U?.41 (PB4)
- net SPI3_NSS: now reaches P1.2 (DAT3), R38.1
- net SPI3_NSS: now also U?.39 (PA15)
- net SPI1_NSS: now reaches U?.12 (PA4)
- net SPI1_NSS: now also R2.1, U5.16 (CS)
- net SPI1_SCK: now reaches U?.13 (PA5)
- net SPI1_SCK: now also U5.17 (SCLK)
- net SPI1_MISO: now reaches U?.14 (PA6)
- net SPI1_MISO: now also R1.2
- net SPI1_MOSI: now reaches U?.15 (PA7)
- net SPI1_MOSI: now also U5.18 (DIN)
- net at U?.22 (PB10): now also R?.1
- net at U?.25 (PB11): now also R?.1
- net SPI2_NSS: now reaches U?.26 (PB12)
- net SPI2_SCK: now reaches U?.27 (PB13)
- net SPI2_MISO: now reaches U?.28 (PB14)
- net SPI2_MOSI: now reaches U?.29 (PB15)
- net NRST renamed G4_NRST
- net G4_NRST: now also J?.1 (Pin_1)
- net RAM_SIO2: no longer names the net of U?.3 (SIO2)
- net RAM_SIO3: no longer names the net of U?.7 (SIO3)
Other:
- note added: "AL_PD"
- note added: "QuadSPI verwenden?"
- note added: "SENSE_+5V"
- note added: "TVS Dioden 3.3V working voltage gegen GND."
- note added: "WOFÜR DIE FAULT PINS??"
- note removed: "OSC-OUT"
- note removed: "SPI?"
- moved on the sheet: C1, C26, C28, C3, C36, C37, C38, C?, D?, FB?, H?, J?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
